File: PCB/Lily58_Pro.sch (KiCad schematic (older format))
At the start: 83 parts, among them J1 LED, J2 4PIN, J3 OLED, P1 i2c_pin, P2 i2c_pin, SW1 SW_PUSH, SW10 SW_PUSH, SW11 SW_PUSH, SW12 SW_PUSH, SW13 SW_PUSH, SW14 SW_PUSH, SW15 SW_PUSH, SW16 SW_PUSH, SW17 SW_PUSH, SW18 SW_PUSH, SW19 SW_PUSH, SW2 SW_PUSH, SW20 SW_PUSH, SW21 SW_PUSH, SW22 SW_PUSH, SW23 SW_PUSH, SW24 SW_PUSH, SW25 SW_PUSH, SW26 SW_PUSH, SW27 SW_PUSH, SW28 SW_PUSH, SW29 SW_PUSH, SW3 SW_PUSH, SW4 SW_PUSH, SW5 SW_PUSH, SW6 SW_PUSH, SW7 SW_PUSH, SW8 SW_PUSH, SW9 SW_PUSH, U1 ProMicro

Commit message: rotary encoder
Parts:
- removed SW25: SW_PUSH, Lily58-footprint:CherryMX_KailhLowProfile_Hotswap, symbol Lily58-cache:SW_PUSH
- added SW25: Rotary_Encoder_Switch, kbd:RotaryEncoder_Alps_EC11E-Switch_Vertical_H20mm-keebio_modified, symbol Device:Rotary_Encoder_Switch
- D1, D10, D11, D12, D13, D14, D15, D16, D17, D18, D19, D2, D20, D21, D22, D23, D24, D25, D26, D27, D28, D29, D3, D4, D5, D6, D7, D8, D9: symbol Lily58-cache:D -> Lily58_Pro-rescue:D-Lily58-cache
- J1: symbol Lily58-cache:LED -> Lily58_Pro-rescue:LED-Lily58-cache
- J2: symbol Lily58-cache:MJ-4PP-9 -> Lily58_Pro-rescue:MJ-4PP-9-Lily58-cache
- J3: symbol Lily58-cache:OLED -> Lily58_Pro-rescue:OLED-Lily58-cache
- P1, P2: symbol Lily58-cache:i2c_pin -> Lily58_Pro-rescue:i2c_pin-Lily58-cache
- R1, R2: symbol Lily58-cache:R -> Lily58_Pro-rescue:R-Lily58-cache
- RSW1: symbol Lily58-cache:SW_RST -> Lily58_Pro-rescue:SW_RST-Lily58-cache
- SW1, SW10, SW11, SW12, SW13, SW14, SW15, SW16, SW17, SW18, SW19, SW2, SW20, SW21, SW22, SW23, SW24, SW26, SW27, SW28, SW29, SW3, SW4, SW5, SW6, SW7, SW8, SW9: footprint Lily58-footprint:CherryMX_KailhLowProfile_Hotswap -> kbd:CherryMX_Choc_Hotswap; symbol Lily58-cache:SW_PUSH -> kbd:SW_PUSH
- TH1, TH2, TH3, TH4, TH5, TH6, TH7: symbol Lily58-cache:HOLE -> Lily58_Pro-rescue:HOLE-Lily58-cache
- U1: symbol Lily58-cache:ProMicro_2 -> Lily58_Pro-rescue:ProMicro_2-Lily58-cache
Connections:
- net labels added: SW25A, SW25B, enc1, enc2
- wire segments 77 -> 86
- no-connect marks 4 -> 2
