File: PCB/Lily58_Pro.kicad_pcb (KiCad board)
At the start: 2 copper layers, 142.5 x 106.3 mm, 83 parts, among them J1 LED, J2 4PIN, J3 OLED, P1 i2c_pin, P2 i2c_pin, SW1 SW_PUSH, SW10 SW_PUSH, SW11 SW_PUSH, SW12 SW_PUSH, SW13 SW_PUSH, SW14 SW_PUSH, SW15 SW_PUSH, SW16 SW_PUSH, SW17 SW_PUSH, SW18 SW_PUSH, SW19 SW_PUSH, SW2 SW_PUSH, SW20 SW_PUSH, SW21 SW_PUSH, SW22 SW_PUSH, SW23 SW_PUSH, SW24 SW_PUSH, SW25 Rotary_Encoder_Switch, SW26 SW_PUSH, SW27 SW_PUSH, SW28 SW_PUSH, SW29 SW_PUSH, SW3 SW_PUSH, SW4 SW_PUSH, SW5 SW_PUSH, SW6 SW_PUSH, SW7 SW_PUSH, SW8 SW_PUSH, SW9 SW_PUSH, U1 ProMicro

Commit message: logo fix
Parts:
- added G***: LOGO, kbd:lily58_logo_Pro, B.Cu at (100.4, 53.6)
- added G***: LOGO, kbd:lily58_logo_Pro, F.Cu at (100.4, 53.6)
- added G***: LOGO, kbd:lily58_logo_2, F.Cu at (97.0, 81.4)
- added G***: LOGO, kbd:lily58_logo_2, B.Cu at (97.0, 81.5)
